File: Amiga_RPI_Drive_Mini_2.3_SMD.brd (EAGLE design)
At the start: 41.9 x 62.2 mm, 45 parts, among them IC1 74LS06D

Commit message: :punch: fixed diodes - v1.1
Parts:
- D1, D2, D3, D4, D5, D7: value B340A -> SB140; device SparkFun-DiscreteSemi:SMA-DIODE -> diode:DO41-10
- LED1: device SparkFun-LED:LED-1206 -> led:LED3MM
- moved D1 19.2 mm to (36.2, 69.8), flipped to the top, turned to 270 degrees
- moved D2 15.9 mm to (33.0, 69.8), turned to 270 degrees
- moved R28 9.25 mm to (37.5, 57.1)
- moved R18 8.64 mm to (12.1, 74.9), turned to 0 degrees
- moved LED1 8.03 mm to (37.5, 61.0)
- moved C1 4.58 mm to (8.89, 67.3), turned to 270 degrees
- moved D3 2.54 mm to (23.5, 69.8), turned to 270 degrees
- moved D4 2.54 mm to (26.7, 69.8), turned to 270 degrees
- moved D5 2.54 mm to (29.8, 69.8), turned to 270 degrees
- moved D7 2.54 mm to (20.3, 69.8), turned to 270 degrees
- moved R2 2.29 mm to (12.1, 72.4)
- moved C2 1.71 mm to (12.1, 57.5), turned to 180 degrees
Connections:
- net GND: now also LED1.K; no longer LED1.C
Routing:
- net GND: track 154.6 -> 95.5 mm, vias 3 -> 2
- net N$8: track 27.9 -> 48.3 mm
- net N$7: track 52.2 -> 70.0 mm, vias 2 -> 3
- net !INDEX: track 26.3 -> 40.5 mm, vias 1 -> 2
- net N$1: track 21.7 -> 32.4 mm, vias 1 -> 2
- net !SEL0: track 54.4 -> 45.7 mm, vias 1 -> 0
- net LED_STEP: track 23.5 -> 15.0 mm
- net !SEL1_IN: track 54.6 -> 57.4 mm
- net !DKRD: track 54.9 -> 52.4 mm
- net VCC: track 112.5 -> 110.3 mm
- net N$5: track 2.58 -> 4.01 mm
- net INDEX_OUT: track 15.3 -> 14.2 mm
- net !CHNG: track 17.6 -> 18.7 mm
- net N$14: track 31.4 -> 30.4 mm
- net N$6: track 28.5 -> 27.7 mm
Other:
- board text added: "smd board v1.1 by stahl"
- board text removed: "smd board v1.0 by stahl"
