File: Amiga_RPI_Drive_Mini_2.3_SMD.sch (EAGLE design)
At the start: 45 parts, among them IC1 74LS06D

Commit message: :punch: fixed diodes - v1.1
Parts:
- D1, D2, D3, D4, D5, D7: value B340A -> SB140; device SparkFun-DiscreteSemi:DIODE-SCHOTTKY-B340A -> diode:SB120
- LED1: device SparkFun-LED:LED-BLUE1206 -> led:LED3MM
Changed lines of the file:
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@@
 <?xml version="1.0" encoding="utf-8"?>
 <!DOCTYPE eagle SYSTEM "eagle.dtd">
-<eagle version="7.7.0">
+<eagle version="7.6.0">
 <drawing>
 <settings>
@@
 <part name="R6" library="SparkFun-Resistors" deviceset="RESISTOR" device="1206" value="1k"/>
 <part name="R7" library="SparkFun-Resistors" deviceset="RESISTOR" device="1206" value="1k"/>
-<part name="D5" library="SparkFun-DiscreteSemi" deviceset="DIODE-SCHOTTKY" device="-B340A" value="B340A"/>
-<part name="D7" library="SparkFun-DiscreteSemi" deviceset="DIODE-SCHOTTKY" device="-B340A" value="B340A"/>
+<part name="D5" library="diode" deviceset="SB120" device="" value="SB140"/>
+<part name="D7" library="diode" deviceset="SB120" device="" value="SB140"/>
 <part name="IC1" library="74xx-eu" deviceset="74*06" device="D" technology="LS" value="74LS06D"/>
 <part name="R21" library="SparkFun-Resistors" deviceset="RESISTOR" device="1206" value="6k8"/>
@@
 <part name="R25" library="SparkFun-Resistors" deviceset="RESISTOR" device="1206" value="6k8"/>
 <part name="R16" library="SparkFun-Resistors" deviceset="RESISTOR" device="1206" value="4k7"/>
-<part name="D1" library="SparkFun-DiscreteSemi" deviceset="DIODE-SCHOTTKY" device="-B340A" value="B340A"/>
-<part name="D2" library="SparkFun-DiscreteSemi" deviceset="DIODE-SCHOTTKY" device="-B340A" value="B340A"/>
+<part name="D1" library="diode" deviceset="SB120" device="" value="SB140"/>
+<part name="D2" library="diode" deviceset="SB120" device="" value="SB140"/>
 <part name="R15" library="SparkFun-Resistors" deviceset="RESISTOR" device="1206" value="10k"/>
 <part name="R14" library="SparkFun-Resistors" deviceset="RESISTOR" device="1206" value="4k7"/>
@@
 <part name="C3" library="SparkFun-Capacitors" deviceset="CAP" device="1206" value="220pf"/>
 <part name="GND4" library="supply1" deviceset="GND" device=""/>
-<part name="D3" library="SparkFun-DiscreteSemi" deviceset="DIODE-SCHOTTKY" device="-B340A" value="B340A"/>
+<part name="D3" library="diode" deviceset="SB120" device="" value="SB140"/>
 <part name="GND2" library="supply1" deviceset="GND" device=""/>
-<part name="D4" library="SparkFun-DiscreteSemi" deviceset="DIODE-SCHOTTKY" device="-B340A" value="B340A"/>
+<part name="D4" library="diode" deviceset="SB120" device="" value="SB140"/>
 <part name="P+5" library="supply1" deviceset="VCC" device=""/>
 <part name="R28" library="SparkFun-Resistors" deviceset="RESISTOR" device="1206" value="330"/>
@@
 <part name="S1" library="switch-dil" deviceset="DS01E" device="" value="SEL1"/>
 <part name="C1" library="rcl" deviceset="CPOL-EU" device="B" value="10uF"/>
-<part name="LED1" library="SparkFun-LED" deviceset="LED-BLUE" device="1206" value="BLUE"/>
+<part name="LED1" library="led" deviceset="LED" device="3MM" value="BLUE"/>
 <part name="BUTTONS" library="mau-pinhead" deviceset="PINHD-1X3" device="" value="gnd | chg | wrt"/>
 <part name="P+2" library="supply1" deviceset="VCC" device=""/>
@@
 <instance part="R6" gate="G$1" x="-137.16" y="78.74" rot="R270"/>
 <instance part="R7" gate="G$1" x="-132.08" y="73.66" rot="R270"/>
-<instance part="D5" gate="G$1" x="-96.52" y="20.32" rot="R90"/>
-<instance part="D7" gate="G$1" x="-88.9" y="20.32" rot="R90"/>
+<instance part="D5" gate="1" x="-96.52" y="20.32" rot="R90"/>
+<instance part="D7" gate="1" x="-88.9" y="20.32" rot="R90"/>
 <instance part="IC1" gate="E" x="-111.76" y="15.24" rot="R180"/>
 <instance part="IC1" gate="C" x="-152.4" y="15.24" rot="R180"/>
@@
 <instance part="IC1" gate="B" x="-137.16" y="-5.08" rot="R180"/>
 <instance part="R16" gate="G$1" x="-93.98" y="2.54" rot="R180"/>
-<instance part="D1" gate="G$1" x="-139.7" y="7.62" rot="R90"/>
-<instance part="D2" gate="G$1" x="-124.46" y="7.62" rot="R90"/>
+<instance part="D1" gate="1" x="-139.7" y="7.62" smashed="yes" rot="R90">
+<attribute name="NAME" x="-140.1826" y="10.16" size="1.778" layer="95" rot="R90"/>
+<attribute name="VALUE" x="-137.3886" y="10.16" size="1.778" layer="96" rot="R90"/>
+</instance>
+<instance part="D2" gate="1" x="-124.46" y="7.62" rot="R90"/>
 <instance part="R15" gate="G$1" x="-99.06" y="-20.32" rot="R180"/>
 <instance part="R14" gate="G$1" x="-101.6" y="22.86" rot="R270"/>
@@
 <instance part="C3" gate="G$1" x="-124.46" y="-25.4"/>
 <instance part="GND4" gate="1" x="-124.46" y="-33.02"/>
-<instance part="D3" gate="G$1" x="-121.92" y="71.12" rot="R270"/>
+<instance part="D3" gate="1" x="-121.92" y="71.12" rot="R270"/>
 <instance part="GND2" gate="1" x="-106.68" y="71.12"/>
-<instance part="D4" gate="G$1" x="-114.3" y="71.12" rot="R270"/>
+<instance part="D4" gate="1" x="-114.3" y="71.12" rot="R270"/>
 <instance part="P+5" gate="VCC" x="-30.48" y="114.3"/>
 <instance part="R28" gate="G$1" x="5.08" y="58.42" rot="MR90"/>
@@
 <wire x1="-88.9" y1="63.5" x2="-88.9" y2="22.86" width="0.1524" layer="91"/>
 <junction x="-88.9" y="63.5"/>
-<pinref part="D7" gate="G$1" pin="C"/>
-<pinref part="D3" gate="G$1" pin="C"/>
+<pinref part="D7" gate="1" pin="C"/>
+<pinref part="D3" gate="1" pin="C"/>
 <junction x="-121.92" y="63.5"/>
 <pinref part="S1" gate="1" pin="2"/>
@@
 </segment>
 <segment>
-<pinref part="D3" gate="G$1" pin="A"/>
+<pinref part="D3" gate="1" pin="A"/>
 <pinref part="GND2" gate="1" pin="GND"/>
 <wire x1="-114.3" y1="76.2" x2="-121.92" y2="76.2" width="0.1524" layer="91"/>
 <wire x1="-121.92" y1="76.2" x2="-121.92" y2="73.66" width="0.1524" layer="91"/>
-<pinref part="D4" gate="G$1" pin="A"/>
+<pinref part="D4" gate="1" pin="A"/>
 <wire x1="-114.3" y1="73.66" x2="-114.3" y2="76.2" width="0.1524" layer="91"/>
 <wire x1="-114.3" y1="76.2" x2="-106.68" y2="76.2" width="0.1524" layer="91"/>
@@
 <wire x1="-96.52" y1="66.04" x2="-96.52" y2="22.86" width="0.1524" layer="91"/>
 <junction x="-96.52" y="66.04"/>
-<pinref part="D5" gate="G$1" pin="C"/>
-<pinref part="D4" gate="G$1" pin="C"/>
+<pinref part="D5" gate="1" pin="C"/>
+<pinref part="D4" gate="1" pin="C"/>
 <junction x="-114.3" y="66.04"/>
 </segment>
@@
 <net name="N$6" class="0">
 <segment>
-<pinref part="D5" gate="G$1" pin="A"/>
-<pinref part="D7" gate="G$1" pin="A"/>
+<pinref part="D5" gate="1" pin="A"/>
+<pinref part="D7" gate="1" pin="A"/>
 <wire x1="-88.9" y1="17.78" x2="-88.9" y2="15.24" width="0.1524" layer="91"/>
 <wire x1="-88.9" y1="15.24" x2="-96.52" y2="15.24" width="0.1524" layer="91"/>
@@
 <pinref part="IC1" gate="E" pin="O"/>
 <pinref part="IC1" gate="C" pin="I"/>
-<pinref part="D1" gate="G$1" pin="C"/>
+<pinref part="D1" gate="1" pin="C"/>
 <wire x1="-124.46" y1="15.24" x2="-132.08" y2="15.24" width="0.1524" layer="91"/>
 <wire x1="-132.08" y1="15.24" x2="-139.7" y2="15.24" width="0.1524" layer="91"/>
 <wire x1="-139.7" y1="10.16" x2="-139.7" y2="15.24" width="0.1524" layer="91"/>
 <wire x1="-139.7" y1="15.24" x2="-142.24" y2="15.24" width="0.1524" layer="91"/>
-<pinref part="D2" gate="G$1" pin="C"/>
+<pinref part="D2" gate="1" pin="C"/>
 <wire x1="-121.92" y1="15.24" x2="-124.46" y2="15.24" width="0.1524" layer="91"/>
 <wire x1="-124.46" y1="15.24" x2="-124.46" y2="10.16" width="0.1524" layer="91"/>
@@
 <pinref part="IC1" gate="A" pin="I"/>
 <wire x1="-99.06" y1="2.54" x2="-139.7" y2="2.54" width="0.1524" layer="91"/>
-<pinref part="D1" gate="G$1" pin="A"/>
+<pinref part="D1" gate="1" pin="A"/>
 <wire x1="-139.7" y1="2.54" x2="-142.24" y2="2.54" width="0.1524" layer="91"/>
 <wire x1="-139.7" y1="5.08" x2="-139.7" y2="2.54" width="0.1524" layer="91"/>
@@
 <pinref part="R15" gate="G$1" pin="2"/>
 <wire x1="-127" y1="-20.32" x2="-124.46" y2="-20.32" width="0.1524" layer="91"/>
-<pinref part="D2" gate="G$1" pin="A"/>
+<pinref part="D2" gate="1" pin="A"/>
 <wire x1="-124.46" y1="-20.32" x2="-106.68" y2="-20.32" width="0.1524" layer="91"/>
 <wire x1="-106.68" y1="-20.32" x2="-104.14" y2="-20.32" width="0.1524" layer="91"/>
